Commit message: esdf and cubit mighty for ground robot

File: urdf/_d435.gazebo.xacro (robot description, xacro)
@@ -14,5 +14,9 @@
                                           infrared1_optical_frame
                                           infrared2_optical_frame
-                                          publish_pointcloud:=true" >
+                                          publish_pointcloud:=true
+                                          color_sensor_rate:=50
+                                          depth_sensor_rate:=100
+                                          depth_plugin_rate:=30.0
+                                          color_plugin_rate:=100.0" >
     <!-- Load parameters to model's main link-->
     <xacro:property name="deg_to_rad" value="0.01745329251994329577" />
@@ -50,5 +54,5 @@
         </camera>
         <always_on>1</always_on>
-        <update_rate>50</update_rate>
+        <update_rate>${color_sensor_rate}</update_rate>
         <visualize>0</visualize>
       </sensor>
@@ -115,5 +119,5 @@
         </camera>
         <always_on>1</always_on>
-        <update_rate>100</update_rate>
+        <update_rate>${depth_sensor_rate}</update_rate>
         <visualize>0</visualize>
       </sensor>
@@ -122,6 +126,6 @@
       <plugin name="${camera_name}" filename="librealsense_gazebo_plugin.so">
         <prefix>${camera_name}</prefix>
-        <depthUpdateRate>30.0</depthUpdateRate>
-        <colorUpdateRate>100.0</colorUpdateRate>
+        <depthUpdateRate>${depth_plugin_rate}</depthUpdateRate>
+        <colorUpdateRate>${color_plugin_rate}</colorUpdateRate>
         <infraredUpdateRate>0.0</infraredUpdateRate>
         <depthTopicName>${topics_ns}/d435/depth/image_raw</depthTopicName>

File: urdf/_d435.urdf.xacro (robot description, xacro)
@@ -9,5 +9,5 @@
   <!--File includes-->
   <xacro:include filename="$(find mighty)/urdf/_d435.gazebo.xacro"/>
-  <xacro:macro name="sensor_d435" params="name:=camera topics_ns range_max_depth parent *origin publish_pointcloud:=true">
+  <xacro:macro name="sensor_d435" params="name:=camera topics_ns range_max_depth parent *origin publish_pointcloud:=true color_sensor_rate:=50 depth_sensor_rate:=100 depth_plugin_rate:=30.0 color_plugin_rate:=100.0">
     <xacro:property name="M_PI" value="3.1415926535897931" />
     <!-- The following values are approximate, and the camera node
@@ -126,5 +126,9 @@
                         infrared1_optical_frame="${name}_left_ir_optical_frame"
                         infrared2_optical_frame="${name}_right_ir_optical_frame"
-                        publish_pointcloud="${publish_pointcloud}"/>
+                        publish_pointcloud="${publish_pointcloud}"
+                        color_sensor_rate="${color_sensor_rate}"
+                        depth_sensor_rate="${depth_sensor_rate}"
+                        depth_plugin_rate="${depth_plugin_rate}"
+                        color_plugin_rate="${color_plugin_rate}"/>
   </xacro:macro>
 </robot>

File: urdf/p3at.urdf.xacro (robot description, xacro)
@@ -22,9 +22,10 @@
   <!-- <xacro:p3at_gazebo_ext name="$(arg namespace)_red_rover" namespace="$(arg namespace)" /> -->
   <xacro:include filename="$(find ros2_livox_simulation)/urdf/mid360.xacro" />
-  <xacro:mid360 name="$(arg namespace)_livox" namespace="$(arg namespace)" parent="base_link" topic="mid360" >
+  <xacro:mid360 name="$(arg namespace)_livox" namespace="$(arg namespace)" parent="base_link" topic="mid360" lidar_update_rate="10" >
     <origin xyz="0 0 1.0" rpy="0 0.3 0"/>
   </xacro:mid360>
   <xacro:include filename="$(find mighty)/urdf/_d435.urdf.xacro" />
-  <xacro:sensor_d435 name="$(arg namespace)_d435" topics_ns="$(arg namespace)" range_max_depth="$(arg d435_range_max_depth)" parent="base_link">
+  <xacro:sensor_d435 name="$(arg namespace)_d435" topics_ns="$(arg namespace)" range_max_depth="$(arg d435_range_max_depth)" parent="base_link"
+                     publish_pointcloud="false" color_sensor_rate="0" depth_sensor_rate="15" depth_plugin_rate="15.0" color_plugin_rate="0.0">
     <origin xyz="1.0 0.0 1.0" rpy="0 0 0"/>
   </xacro:sensor_d435>

File: urdf/sonar_sensor.urdf.xacro (robot description, xacro)
@@ -31,6 +31,6 @@
         <pose>0 0 0 0 0 0</pose>
         <always_on>true</always_on>
-        <visualize>true</visualize>
-        <update_rate>40</update_rate>
+        <visualize>false</visualize>
+        <update_rate>10</update_rate>
         <ray>
           <scan>
